File: p1+_drive/KiCAD/p1+_drive.kicad_sch (KiCad schematic)
At the start: 16 parts, among them J1 SD_Card_Device, SW1 interface

Commit message: Ajout d'une RAM 128KB 23LC1024 au circuit du p1+_drive
Parts:
- removed SW1: interface, symbol Switch:SW_SPST
- added J2: interface, symbol Connector:Conn_01x02_Pin
Connections:
- net GND: now also J2.2 (Pin_2)
- net at U1.11 (PB5/AIN5): now also J2.1 (Pin_1)
Other:
- note added: "J2"
- note removed: "SW1"
Changed lines of the file:
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@@
 	)
 	(no_connect
+		(at 113.03 123.19)
+	)
+	(no_connect
 		(at 113.03 95.25)
 	)
@@
 	)
 	(no_connect
-		(at 113.03 118.11)
-	)
-	(no_connect
 		(at 113.03 97.79)
 	)
@@
 	(wire
 		(pts
+			(xy 90.17 118.11) (xy 113.03 118.11)
+		)
+		(stroke
+			(width 0)
+			(type default)
+		)
+	)
+	(wire
+		(pts
 			(xy 170.18 157.48) (xy 171.45 157.48)
 		)
@@
 	(wire
 		(pts
-			(xy 96.52 123.19) (xy 113.03 123.19)
-		)
-		(stroke
-			(width 0)
-			(type default)
-		)
-	)
-	(wire
-		(pts
 			(xy 144.78 113.03) (xy 147.32 113.03)
 		)
@@
 	(wire
 		(pts
-			(xy 81.28 123.19) (xy 86.36 123.19)
-		)
-		(stroke
-			(width 0)
-			(type default)
-		)
-	)
-	(wire
-		(pts
 			(xy 106.68 168.91) (xy 115.57 168.91)
 		)
@@
 		)
 	)
-	(text "SW1"
+	(text "J2"
 		(exclude_from_sim no)
 		(at 84.836 133.096 0)
@@
 	)
 	(symbol
-		(lib_id "power:GND")
-		(at 81.28 123.19 0)
+		(lib_id "Device:C")
+		(at 115.57 165.1 0)
 		(unit 1)
 		(exclude_from_sim no)
@@
 		(on_board yes)
 		(dnp no)
-		(fields_autoplaced yes)
-		(property "Reference" "#PWR012"
-			(at 81.28 129.54 0)
+		(property "Reference" "C3"
+			(at 115.57 163.068 0)
 			(effects
 				(font
 					(size 1.27 1.27)
 				)
-				(hide yes)
+				(justify left)
 			)
 		)
-		(property "Value" "GND"
-			(at 81.28 128.27 0)
+		(property "Value" "100nF"
+			(at 115.57 167.386 0)
 			(effects
 				(font
 					(size 1.27 1.27)
 				)
+				(justify left)
 			)
 		)
 		(property "Footprint" ""
-			(at 81.28 123.19 0)
+			(at 116.5352 168.91 0)
 			(effects
 				(font
@@
 			)
 		)
-		(property "Datasheet" ""
-			(at 81.28 123.19 0)
+		(property "Datasheet" "~"
+			(at 115.57 165.1 0)
 			(effects
 				(font
@@
 			)
 		)
-		(property "Description" "Power symbol creates a global label with name \"GND\" , ground"
-			(at 81.28 123.19 0)
+		(property "Description" "Unpolarized capacitor"
+			(at 115.57 165.1 0)
 			(effects
 				(font
@@
 		(pin "1"
 		)
+		(pin "2"
+		)
 		(instances
-			(project "p1+_drive"
+			(project ""
 				(path "/10ea552d-8990-4500-8ec9-fced7d5632e2"
-					(reference "#PWR012")
+					(reference "C3")
 					(unit 1)
 				)
@@
 	)
 	(symbol
-		(lib_id "Device:C")
-		(at 115.57 165.1 0)
+		(lib_id "power:GND")
+		(at 218.44 113.03 0)
 		(unit 1)
 		(exclude_from_sim no)
@@
 		(on_board yes)
 		(dnp no)
-		(property "Reference" "C3"
-			(at 115.57 163.068 0)
+		(fields_autoplaced yes)
+		(property "Reference" "#PWR05"
+			(at 218.44 119.38 0)
 			(effects
 				(font
 					(size 1.27 1.27)
 				)
-				(justify left)
+				(hide yes)
 			)
 		)
-		(property "Value" "100nF"
-			(at 115.57 167.386 0)
+		(property "Value" "GND"
+			(at 218.44 118.11 0)
 			(effects
 				(font
 					(size 1.27 1.27)
 				)
-				(justify left)
 			)
 		)
 		(property "Footprint" ""
-			(at 116.5352 168.91 0)
+			(at 218.44 113.03 0)
 			(effects
 				(font
@@
 			)
 		)
-		(property "Datasheet" "~"
-			(at 115.57 165.1 0)
+		(property "Datasheet" ""
+			(at 218.44 113.03 0)
 			(effects
 				(font
@@
 			)
 		)
-		(property "Description" "Unpolarized capacitor"
-			(at 115.57 165.1 0)
+		(property "Description" "Power symbol creates a global label with name \"GND\" , ground"
+			(at 218.44 113.03 0)
 			(effects
 				(font
@@
 		(pin "1"
 		)
-		(pin "2"
-		)
 		(instances
-			(project ""
+			(project "p1+_drive"
 				(path "/10ea552d-8990-4500-8ec9-fced7d5632e2"
-					(reference "C3")
+					(reference "#PWR05")
 					(unit 1)
 				)
@@
 	(symbol
 		(lib_id "power:GND")
-		(at 218.44 113.03 0)
+		(at 90.17 120.65 0)
 		(unit 1)
 		(exclude_from_sim no)
@@
 		(on_board yes)
 		(dnp no)
-		(fields_autoplaced yes)
-		(property "Reference" "#PWR05"
-			(at 218.44 119.38 0)
+		(property "Reference" "#PWR08"
+			(at 90.17 127 0)
 			(effects
 				(font
@@
 		)
 		(property "Value" "GND"
-			(at 218.44 118.11 0)
+			(at 90.17 123.19 90)
 			(effects
 				(font
 					(size 1.27 1.27)
 				)
+				(justify right)
 			)
 		)
 		(property "Footprint" ""
-			(at 218.44 113.03 0)
+			(at 90.17 120.65 0)
 			(effects
 				(font
@@
 		)
 		(property "Datasheet" ""
-			(at 218.44 113.03 0)
+			(at 90.17 120.65 0)
 			(effects
 				(font
@@
 		)
 		(property "Description" "Power symbol creates a global label with name \"GND\" , ground"
-			(at 218.44 113.03 0)
+			(at 90.17 120.65 0)
 			(effects
 				(font
@@
 			(project "p1+_drive"
 				(path "/10ea552d-8990-4500-8ec9-fced7d5632e2"
-					(reference "#PWR05")
+					(reference "#PWR08")
 					(unit 1)
 				)
@@
 	)
 	(symbol
+		(lib_id "Connector:Conn_01x02_Pin")
+		(at 85.09 118.11 0)
+		(unit 1)
+		(exclude_from_sim no)
+		(in_bom yes)
+		(on_board yes)
+		(dnp no)
+		(fields_autoplaced yes)
+		(property "Reference" "J2"
+			(at 85.725 113.03 0)
+			(effects
+				(font
+					(size 1.27 1.27)
+				)
+			)
+		)
+		(property "Value" "interface"
+			(at 85.725 115.57 0)
+			(effects
+				(font
+					(size 1.27 1.27)
+				)
+			)
+		)
+		(property "Footprint" ""
+			(at 85.09 118.11 0)
+			(effects
+				(font
+					(size 1.27 1.27)
+				)
+				(hide yes)
+			)
+		)
+		(property "Datasheet" "~"
+			(at 85.09 118.11 0)
+			(effects
+				(font
+					(size 1.27 1.27)
+				)
+				(hide yes)
+			)
+		)
+		(property "Description" "Generic connector, single row, 01x02, script generated"
+			(at 85.09 118.11 0)
+			(effects
+				(font
+					(size 1.27 1.27)
+				)
+				(hide yes)
+			)
+		)
+		(pin "2"
+		)
+		(pin "1"
+		)
+		(instances
+			(project ""
+				(path "/10ea552d-8990-4500-8ec9-fced7d5632e2"
+					(reference "J2")
+					(unit 1)
+				)
+			)
+		)
+	)
+	(symbol
 		(lib_id "STM8S207K8T:STM8S207K8T")
 		(at 128.27 111.76 0)
@@
 					(unit 1)
 				)
-			)
-		)
-	)
-	(symbol
-		(lib_id "Switch:SW_SPST")
-		(at 91.44 123.19 0)
-		(unit 1)
-		(exclude_from_sim no)
-		(in_bom yes)
-		(on_board yes)
-		(dnp no)
-		(property "Reference" "SW1"
-			(at 91.694 119.38 0)
-			(effects
-				(font
-					(size 1.27 1.27)
-				)
-			)
-		)
-		(property "Value" "interface"
-			(at 91.694 125.222 0)
-			(effects
-				(font
-					(size 1.27 1.27)
-				)
-			)
-		)
-		(property "Footprint" ""
-			(at 91.44 123.19 0)
-			(effects
-				(font
-					(size 1.27 1.27)
-				)
-				(hide yes)
-			)
-		)
-		(property "Datasheet" "~"
-			(at 91.44 123.19 0)
-			(effects
-				(font
-					(size 1.27 1.27)
-				)
-				(hide yes)
-			)
-		)
-		(property "Description" "Single Pole Single Throw (SPST) switch"
-			(at 91.44 123.19 0)
-			(effects
-				(font
-					(size 1.27 1.27)
-				)
-				(hide yes)
-			)
-		)
-		(pin "1"
-		)
-		(pin "2"
-		)
-		(instances
-			(project ""
-				(path "/10ea552d-8990-4500-8ec9-fced7d5632e2"
-					(reference "SW1")
-					(unit 1)
-				)
