File: KiCAD/pomme-1+/mémoire.kicad_sch (KiCad schematic)
At the start: 14 parts

Commit message: Modification de la conception du pomme 1+ Ajout d'un PIA W65C22 à la carte périphériques Ajout d'un régulateur de tension 3.3V à l'alimentation
Connections:
- net +5V is gone; now on net Vcc: U11.14 (VDD), U5.27 (~WE), U5.28 (VCC), U6.27 (~WE), U6.28 (VCC), U8.28 (VCC)
- net Vcc: now reaches C10.1, C11.1, C12.1, C13.1, C14.1, C23.1, C24.1, C25.1, C26.1, C9.1
- net READ renamed READ/~{WRITE}
Other:
- note added: "pomme 1+ memory board"
- moved on the sheet: U11E
Changed lines of the file:
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@@
 	(wire
 		(pts
-			(xy 19.05 142.24) (xy 19.05 144.78)
+			(xy 27.94 142.24) (xy 27.94 144.78)
 		)
 		(stroke
@@
 		)
 	)
+	(text "pomme 1+\nmemory board"
+		(exclude_from_sim no)
+		(at 179.578 173.482 0)
+		(effects
+			(font
+				(size 3.81 3.81)
+			)
+			(justify left)
+		)
+	)
 	(text "0xE000-0xFFFF"
 		(exclude_from_sim no)
@@
 		)
 	)
-	(global_label "+5V"
+	(global_label "Vcc"
 		(shape input)
 		(at 179.07 118.11 0)
@@
 		)
 		(property "Intersheetrefs" "${INTERSHEET_REFS}"
-			(at 184.5543 118.11 0)
+			(at 184.0706 118.11 0)
+			(effects
+				(font
+					(size 1.27 1.27)
+				)
+				(justify left)
+				(hide yes)
+			)
+		)
+	)
+	(global_label "Vcc"
+		(shape input)
+		(at 97.79 172.72 90)
+		(fields_autoplaced yes)
+		(effects
+			(font
+				(size 1.016 1.016)
+			)
+			(justify left)
+		)
+		(property "Intersheetrefs" "${INTERSHEET_REFS}"
+			(at 97.79 167.7194 90)
 			(effects
 				(font
@@
 		)
 	)
-	(global_label "+5V"
+	(global_label "Vcc"
 		(shape input)
 		(at 182.88 69.85 0)
@@
 		)
 		(property "Intersheetrefs" "${INTERSHEET_REFS}"
-			(at 188.3643 69.85 0)
+			(at 187.8806 69.85 0)
 			(effects
 				(font
@@
 		)
 	)
-	(global_label "READ"
+	(global_label "READ{slash}~{WRITE}"
 		(shape input)
 		(at 179.07 120.65 0)
@@
 		)
 		(property "Intersheetrefs" "${INTERSHEET_REFS}"
-			(at 185.28 120.65 0)
+			(at 190.6986 120.65 0)
 			(effects
 				(font
@@
 		)
 	)
-	(global_label "+5V"
+	(global_label "Vcc"
 		(shape input)
 		(at 182.88 22.86 0)
@@
 		)
 		(property "Intersheetrefs" "${INTERSHEET_REFS}"
-			(at 188.3643 22.86 0)
+			(at 187.8806 22.86 0)
 			(effects
 				(font
@@
 		)
 	)
-	(global_label "+5V"
+	(global_label "Vcc"
 		(shape input)
-		(at 19.05 142.24 90)
+		(at 27.94 142.24 90)
 		(fields_autoplaced yes)
 		(effects
@@
 		)
 		(property "Intersheetrefs" "${INTERSHEET_REFS}"
-			(at 19.05 136.7557 90)
+			(at 27.94 137.2394 90)
 			(effects
 				(font
@@
 	(symbol
 		(lib_id "power:GND")
-		(at 19.05 160.02 0)
+		(at 27.94 160.02 0)
 		(unit 1)
 		(exclude_from_sim no)
@@
 		(fields_autoplaced yes)
 		(property "Reference" "#PWR019"
-			(at 19.05 166.37 0)
+			(at 27.94 166.37 0)
 			(effects
 				(font
@@
 		)
 		(property "Value" "GND"
-			(at 19.05 165.1 0)
+			(at 27.94 165.1 0)
 			(effects
 				(font
@@
 		)
 		(property "Footprint" ""
-			(at 19.05 160.02 0)
+			(at 27.94 160.02 0)
 			(effects
 				(font
@@
 		)
 		(property "Datasheet" ""
-			(at 19.05 160.02 0)
+			(at 27.94 160.02 0)
 			(effects
 				(font
@@
 		)
 		(property "Description" "Power symbol creates a global label with name \"GND\" , ground"
-			(at 19.05 160.02 0)
+			(at 27.94 160.02 0)
 			(effects
 				(font
@@
 		(on_board yes)
 		(dnp no)
-		(fields_autoplaced yes)
 		(property "Reference" "U11"
-			(at 57.658 132.08 0)
+			(at 57.404 134.366 0)
 			(effects
 				(font
@@
 	(symbol
 		(lib_id "my74HCxx:SN74HC08N")
-		(at 19.05 152.4 0)
+		(at 27.94 152.4 0)
 		(unit 5)
 		(exclude_from_sim no)
@@
 		(fields_autoplaced yes)
 		(property "Reference" "U11"
-			(at 22.86 151.7649 0)
+			(at 31.75 151.7649 0)
 			(effects
 				(font
@@
 		)
 		(property "Value" "~"
-			(at 22.86 153.67 0)
+			(at 31.75 153.67 0)
 			(effects
 				(font
@@
 		)
 		(property "Footprint" ""
-			(at 19.05 152.4 0)
+			(at 27.94 152.4 0)
 			(effects
 				(font
@@
 		)
 		(property "Datasheet" ""
-			(at 19.05 152.4 0)
+			(at 27.94 152.4 0)
 			(effects
 				(font
@@
 		)
 		(property "Description" ""
-			(at 19.05 152.4 0)
+			(at 27.94 152.4 0)
 			(effects
 				(font
@@
 		(on_board yes)
 		(dnp no)
-		(fields_autoplaced yes)
 		(property "Reference" "U11"
-			(at 57.4675 146.05 0)
-			(effects
-				(font
+			(at 57.404 147.828 0)
+			(effects
+				(font

Commit message: Modification documents
Parts:
- renumbered C9 to C26, C10 to C27, C11 to C28, C12 to C29, C13 to C30, C14 to C31, C23 to C32, C24 to C33, C25 to C34, C26 to C35, U11 to U12, U5 to U13, U6 to U14, U8 to U15
Changed lines of the file:
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@@
 		(dnp no)
 		(fields_autoplaced yes)
-		(property "Reference" "C25"
+		(property "Reference" "C34"
 			(at 154.94 175.2599 0)
 			(effects
@@
 			(project "pomme-1.5"
 				(path "/46a37b86-f1f5-4cd9-9809-f219c84ab6f2/5cafbe69-2de4-4de2-951a-877394ff761e"
-					(reference "C25")
+					(reference "C34")
 					(unit 1)
 				)
@@
 		(dnp no)
 		(fields_autoplaced yes)
-		(property "Reference" "C13"
+		(property "Reference" "C30"
 			(at 93.98 174.3709 0)
 			(effects
@@
 			(project "pomme-1.5"
 				(path "/46a37b86-f1f5-4cd9-9809-f219c84ab6f2/5cafbe69-2de4-4de2-951a-877394ff761e"
-					(reference "C13")
+					(reference "C30")
 					(unit 1)
 				)
@@
 		(on_board yes)
 		(dnp no)
-		(property "Reference" "U11"
+		(property "Reference" "U12"
 			(at 187.96 93.98 0)
 			(effects
@@
 			(project ""
 				(path "/46a37b86-f1f5-4cd9-9809-f219c84ab6f2/5cafbe69-2de4-4de2-951a-877394ff761e"
-					(reference "U11")
+					(reference "U12")
 					(unit 1)
 				)
@@
 		(dnp no)
 		(fields_autoplaced yes)
-		(property "Reference" "#PWR019"
+		(property "Reference" "#PWR027"
 			(at 27.94 166.37 0)
 			(effects
@@
 			(project ""
 				(path "/46a37b86-f1f5-4cd9-9809-f219c84ab6f2/5cafbe69-2de4-4de2-951a-877394ff761e"
-					(reference "#PWR019")
+					(reference "#PWR027")
 					(unit 1)
 				)
@@
 		(on_board yes)
 		(dnp no)
-		(property "Reference" "#PWR08"
+		(property "Reference" "#PWR028"
 			(at 153.67 67.31 0)
 			(effects
@@
 			(project "pomme-1.5"
 				(path "/46a37b86-f1f5-4cd9-9809-f219c84ab6f2/5cafbe69-2de4-4de2-951a-877394ff761e"
-					(reference "#PWR08")
+					(reference "#PWR028")
 					(unit 1)
 				)
@@
 		(on_board yes)
 		(dnp no)
-		(property "Reference" "U11"
+		(property "Reference" "U12"
 			(at 188.214 46.99 0)
 			(effects
@@
 			(project ""
 				(path "/46a37b86-f1f5-4cd9-9809-f219c84ab6f2/5cafbe69-2de4-4de2-951a-877394ff761e"
-					(reference "U11")
+					(reference "U12")
 					(unit 2)
 				)
@@
 		(dnp no)
 		(fields_autoplaced yes)
-		(property "Reference" "C9"
+		(property "Reference" "C26"
 			(at 20.32 174.3709 0)
 			(effects
@@
 			(project "pomme-1.5"
 				(path "/46a37b86-f1f5-4cd9-9809-f219c84ab6f2/5cafbe69-2de4-4de2-951a-877394ff761e"
-					(reference "C9")
+					(reference "C26")
 					(unit 1)
 				)
@@
 		(dnp no)
 		(fields_autoplaced yes)
-		(property "Reference" "C11"
+		(property "Reference" "C28"
 			(at 57.15 174.3709 0)
 			(effects
@@
 			(project "pomme-1.5"
 				(path "/46a37b86-f1f5-4cd9-9809-f219c84ab6f2/5cafbe69-2de4-4de2-951a-877394ff761e"
-					(reference "C11")
+					(reference "C28")
 					(unit 1)
 				)
@@
 		(dnp no)
 		(fields_autoplaced yes)
-		(property "Reference" "C12"
+		(property "Reference" "C29"
 			(at 76.2 174.3709 0)
 			(effects
@@
 			(project "pomme-1.5"
 				(path "/46a37b86-f1f5-4cd9-9809-f219c84ab6f2/5cafbe69-2de4-4de2-951a-877394ff761e"
-					(reference "C12")
+					(reference "C29")
 					(unit 1)
 				)
@@
 		(dnp no)
 		(fields_autoplaced yes)
-		(property "Reference" "C24"
+		(property "Reference" "C33"
 			(at 140.97 175.2599 0)
 			(effects
@@
 			(project "pomme-1.5"
 				(path "/46a37b86-f1f5-4cd9-9809-f219c84ab6f2/5cafbe69-2de4-4de2-951a-877394ff761e"
-					(reference "C24")
+					(reference "C33")
 					(unit 1)
 				)
@@
 		(on_board yes)
 		(dnp no)
-		(property "Reference" "U11"
+		(property "Reference" "U12"
 			(at 57.404 134.366 0)
 			(effects
@@
 			(project ""
 				(path "/46a37b86-f1f5-4cd9-9809-f219c84ab6f2/5cafbe69-2de4-4de2-951a-877394ff761e"
-					(reference "U11")
+					(reference "U12")
 					(unit 3)
 				)
@@
 		(dnp no)
 		(fields_autoplaced yes)
-		(property "Reference" "C14"
+		(property "Reference" "C31"
 			(at 111.76 174.3709 0)
 			(effects
@@
 			(project "pomme-1.5"
 				(path "/46a37b86-f1f5-4cd9-9809-f219c84ab6f2/5cafbe69-2de4-4de2-951a-877394ff761e"
-					(reference "C14")
+					(reference "C31")
 					(unit 1)
 				)
@@
 		(dnp no)
 		(fields_autoplaced yes)
-		(property "Reference" "U11"
+		(property "Reference" "U12"
 			(at 31.75 151.7649 0)
 			(effects
@@
 			(project ""
 				(path "/46a37b86-f1f5-4cd9-9809-f219c84ab6f2/5cafbe69-2de4-4de2-951a-877394ff761e"
-					(reference "U11")
+					(reference "U12")
 					(unit 5)
 				)
@@
 		(on_board yes)
 		(dnp no)
-		(property "Reference" "#PWR013"
+		(property "Reference" "#PWR030"
 			(at 156.21 165.1 0)
 			(effects
@@
 			(project "pomme-1.5"
 				(path "/46a37b86-f1f5-4cd9-9809-f219c84ab6f2/5cafbe69-2de4-4de2-951a-877394ff761e"
-					(reference "#PWR013")
+					(reference "#PWR030")
 					(unit 1)
 				)
@@
 		(on_board yes)
 		(dnp no)
-		(property "Reference" "U6"
+		(property "Reference" "U14"
 			(at 163.83 67.564 0)
 			(effects
@@
 			(project "pomme-1.5"
 				(path "/46a37b86-f1f5-4cd9-9809-f219c84ab6f2/5cafbe69-2de4-4de2-951a-877394ff761e"
-					(reference "U6")
+					(reference "U14")
 					(unit 1)
 				)
@@
 		(dnp no)
 		(fields_autoplaced yes)
-		(property "Reference" "C26"
+		(property "Reference" "C35"
 			(at 170.18 175.2599 0)
 			(effects
@@
 			(project "pomme-1.5"
 				(path "/46a37b86-f1f5-4cd9-9809-f219c84ab6f2/5cafbe69-2de4-4de2-951a-877394ff761e"
-					(reference "C26")
+					(reference "C35")
 					(unit 1)
 				)
@@
 		(dnp no)
 		(fields_autoplaced yes)
-		(property "Reference" "C23"
+		(property "Reference" "C32"
 			(at 128.27 175.2599 0)
 			(effects
@@
 			(project "pomme-1.5"
 				(path "/46a37b86-f1f5-4cd9-9809-f219c84ab6f2/5cafbe69-2de4-4de2-951a-877394ff761e"
-					(reference "C23")
+					(reference "C32")
 					(unit 1)
 				)
@@
 		(dnp no)
 		(fields_autoplaced yes)
-		(property "Reference" "C10"
+		(property "Reference" "C27"
 			(at 39.37 174.3709 0)
 			(effects
@@
 			(project "pomme-1.5"
 				(path "/46a37b86-f1f5-4cd9-9809-f219c84ab6f2/5cafbe69-2de4-4de2-951a-877394ff761e"
-					(reference "C10")
+					(reference "C27")
 					(unit 1)
 				)
@@
 		(on_board yes)
 		(dnp no)
-		(property "Reference" "U8"
+		(property "Reference" "U15"
 			(at 166.37 115.57 0)
 			(effects
@@
 			(project "pomme-1.5"
 				(path "/46a37b86-f1f5-4cd9-9809-f219c84ab6f2/5cafbe69-2de4-4de2-951a-877394ff761e"
-					(reference "U8")
+					(reference "U15")
 					(unit 1)
 				)
@@
 		(on_board yes)
 		(dnp no)
-		(property "Reference" "#PWR09"
+		(property "Reference" "#PWR029"
 			(at 153.67 114.3 0)
 			(effects
@@
 			(project "pomme-1.5"
 				(path "/46a37b86-f1f5-4cd9-9809-f219c84ab6f2/5cafbe69-2de4-4de2-951a-877394ff761e"
-					(reference "#PWR09")
+					(reference "#PWR029")
 					(unit 1)
 				)
@@
 		(on_board yes)
 		(dnp no)
-		(property "Reference" "U5"
+		(property "Reference" "U13"
 			(at 163.83 20.574 0)
 			(effects
@@
 			(project "pomme-1.5"
 				(path "/46a37b86-f1f5-4cd9-9809-f219c84ab6f2/5cafbe69-2de4-4de2-951a-877394ff761e"
-					(reference "U5")
+					(reference "U13")
 					(unit 1)
 				)
@@
 		(on_board yes)
 		(dnp no)
-		(property "Reference" "U11"
+		(property "Reference" "U12"
 			(at 57.404 147.828 0)
 			(effects
@@
 			(project ""
 				(path "/46a37b86-f1f5-4cd9-9809-f219c84ab6f2/5cafbe69-2de4-4de2-951a-877394ff761e"
-					(reference "U11")
+					(reference "U12")
 					(unit 4)
 				)

Commit message: Modification au circuit du pomme-1+ ajout d'une seconde EEPROM (U13) 0xC000...0xDFFF. Celle-ci peut-être programmée dans le circuit.
Parts:
- added R16, R17: 4K7, symbol Device:R
Connections:
- net GND: now also C26.2, C27.2, C28.2, C29.2, C30.2, C31.2, C32.2, C33.2, C34.2, C35.2
- net Vcc: now also R16.1, R17.1; no longer U13.27 (~WE)
- net U13_~{BUSY}: now reaches U13.1 (NC)
- net U13_~{BUSY}: now also R17.2
- new net U13_~{WE}: R16.2, U13.27 (~WE)

Commit message: Modification au circuit pour supprimer le polling de la pin 1 de U13, car ça ne fonctionne pas bien. La solution logiciel est plus fiable.
Parts:
- removed R17: 4K7, symbol Device:R
Connections:
- net U13_~{BUSY}: no longer names the net of U13.1 (NC)
- no-connect marks 0 -> 2
Changed lines of the file:
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@@
 	)
 	(junction
-		(at 182.88 17.78)
-		(diameter 0)
-		(color 0 0 0 0)
-	)
-	(junction
 		(at 116.84 180.34)
 		(diameter 0)
@@
 	)
 	(junction
-		(at 142.24 22.86)
-		(diameter 0)
-		(color 0 0 0 0)
-	)
-	(junction
 		(at 90.17 172.72)
 		(diameter 0)
@@
 		(color 0 0 0 0)
 	)
+	(no_connect
+		(at 153.67 22.86)
+	)
+	(no_connect
+		(at 173.99 27.94)
+	)
 	(bus_entry
 		(at 153.67 125.73)
@@
 		)
 	)
-	(wire
-		(pts
-			(xy 151.13 22.86) (xy 153.67 22.86)
-		)
-		(stroke
-			(width 0)
-			(type default)
-		)
-	)
 	(bus
 		(pts
@@
 	(wire
 		(pts
-			(xy 182.88 15.24) (xy 182.88 17.78)
-		)
-		(stroke
-			(width 0)
-			(type default)
-		)
-	)
-	(wire
-		(pts
 			(xy 35.56 180.34) (xy 53.34 180.34)
 		)
@@
 	(wire
 		(pts
-			(xy 142.24 22.86) (xy 151.13 22.86)
-		)
-		(stroke
-			(width 0)
-			(type default)
-		)
-	)
-	(wire
-		(pts
 			(xy 176.53 38.1) (xy 179.07 38.1)
 		)
@@
 		)
 	)
-	(wire
-		(pts
-			(xy 139.7 22.86) (xy 142.24 22.86)
-		)
-		(stroke
-			(width 0)
-			(type default)
-		)
-	)
 	(bus
 		(pts
@@
 		)
 	)
-	(wire
-		(pts
-			(xy 142.24 15.24) (xy 182.88 15.24)
-		)
-		(stroke
-			(width 0)
-			(type default)
-		)
-	)
 	(bus
 		(pts
@@
 		)
 	)
-	(global_label "U13_~{BUSY}"
-		(shape output)
-		(at 139.7 22.86 180)
-		(fields_autoplaced yes)
-		(effects
-			(font
-				(size 1.27 1.27)
-			)
-			(justify right)
-		)
-		(property "Intersheetrefs" "${INTERSHEET_REFS}"
-			(at 127.0991 22.86 0)
-			(effects
-				(font
-					(size 1.27 1.27)
-				)
-				(justify right)
-				(hide yes)
-			)
-		)
-	)
 	(global_label "~{OE}"
 		(shape input)
@@
 					(unit 1)
 				)
-			)
-		)
-	)
-	(symbol
-		(lib_id "Device:R")
-		(at 142.24 19.05 0)
-		(unit 1)
-		(exclude_from_sim no)
-		(in_bom yes)
-		(on_board yes)
-		(dnp no)
-		(fields_autoplaced yes)
-		(property "Reference" "R17"
-			(at 144.78 17.7799 0)
-			(effects
-				(font
-					(size 1.27 1.27)
-				)
-				(justify left)
-			)
-		)
-		(property "Value" "4K7"
-			(at 144.78 20.3199 0)
-			(effects
-				(font
-					(size 1.27 1.27)
-				)
-				(justify left)
-			)
-		)
-		(property "Footprint" ""
-			(at 140.462 19.05 90)
-			(effects
-				(font
-					(size 1.27 1.27)
-				)
-				(hide yes)
-			)
-		)
-		(property "Datasheet" "~"
-			(at 142.24 19.05 0)
-			(effects
-				(font
-					(size 1.27 1.27)
-				)
-				(hide yes)
-			)
-		)
-		(property "Description" "Resistor"
-			(at 142.24 19.05 0)
-			(effects
-				(font
-					(size 1.27 1.27)
-				)
-				(hide yes)
-			)
-		)
-		(pin "2"
-		)
-		(pin "1"
-		)
-		(instances
-			(project "pomme-1.5"
-				(path "/46a37b86-f1f5-4cd9-9809-f219c84ab6f2/5cafbe69-2de4-4de2-951a-877394ff761e"
-					(reference "R17")
-					(unit 1)
-				)
